File: Connectors.kicad_sch (KiCad schematic)
At the start: 41 parts, among them J1 DB15, J2 DB15, J4 HEADER_16, P1 Conn_GPS, P2 Conn_BMP280, P3 I2C_EXT, P4 I2C_EXT, P5 CONN_01X06, P6 CONN_01X04

Commit message: Agrego la version modificada para Mario de Ecuador, con vias mas grandes
Parts:
- C11: symbol lago_sch-rescue:C_Small -> lago_sch-rescue:C_Small-lago_sch-rescue
- D5, D6: symbol lago_sch-rescue:ZENERsmall -> lago_sch-rescue:ZENERsmall-lago_sch-rescue
- GS1, GS2, GS3, GS4: symbol lago_sch-rescue:GS2 -> lago_sch-rescue:GS2-lago_sch-rescue
- J1, J2: symbol lago_sch-rescue:DB15 -> lago_sch-rescue:DB15-lago_sch-rescue
- J4: symbol lago_sch-rescue:HEADER_16 -> lago_sch-rescue:HEADER_16-lago_sch-rescue
- JP5: symbol lago_sch-rescue:Jumper_NO_Small -> lago_sch-rescue:Jumper_NO_Small-lago_sch-rescue
- L10, L11, L12, L13, L14, L15, L16, L17, L18, L7, L8, L9: symbol lago_sch-rescue:L -> lago_sch-rescue:L-lago_sch-rescue
- P1: symbol lago_sch-rescue:CONN_01X08 -> lago_sch-rescue:CONN_01X08-lago_sch-rescue
- P2, P3, P4, P6: symbol lago_sch-rescue:CONN_01X04 -> lago_sch-rescue:CONN_01X04-lago_sch-rescue
- P5: symbol lago_sch-rescue:CONN_01X06 -> lago_sch-rescue:CONN_01X06-lago_sch-rescue
- R13, R14, R15, R16: symbol lago_sch-rescue:R -> lago_sch-rescue:R-lago_sch-rescue
- R17, R18, R19, R20: symbol lago_sch-rescue:R_Small -> lago_sch-rescue:R_Small-lago_sch-rescue
- RP_E1, RP_E2: symbol lago_sch-rescue:CONN_02X13 -> lago_sch-rescue:CONN_02X13-lago_sch-rescue
- W10, W9: symbol lago_sch-rescue:TEST_1P -> lago_sch-rescue:TEST_1P-lago_sch-rescue
