File: lago_sch.kicad_sch (KiCad schematic)
At the start: 31 parts, among them U1 LM324

Commit message: Agrego la version modificada para Mario de Ecuador, con vias mas grandes
Parts:
- C1, C2, C3, C4: symbol lago_sch-rescue:cap -> lago_sch-rescue:cap-lago_sch-rescue
- C10: symbol lago_sch-rescue:CP1 -> lago_sch-rescue:CP1-lago_sch-rescue
- C5, C6, C7, C8, C9: symbol lago_sch-rescue:C -> lago_sch-rescue:C-lago_sch-rescue
- D1, D2, D3, D4: symbol lago_sch-rescue:ZENERsmall -> lago_sch-rescue:ZENERsmall-lago_sch-rescue
- R1, R10, R11, R12, R2, R3, R4, R5, R6, R7, R8, R9: symbol lago_sch-rescue:R -> lago_sch-rescue:R-lago_sch-rescue
- U1: symbol lago_sch-rescue:LM324 -> lago_sch-rescue:LM324-lago_sch-rescue
- W5, W6, W7, W8: symbol lago_sch-rescue:TEST_1P -> lago_sch-rescue:TEST_1P-lago_sch-rescue
