File: power.kicad_sch (KiCad schematic)
At the start: 58 parts, among them J3 BARREL_JACK, U2 LM2596, U3 LT8471

Commit message: Agrego la version modificada para Mario de Ecuador, con vias mas grandes
Parts:
- C12, C22: symbol lago_sch-rescue:CP -> lago_sch-rescue:CP-lago_sch-rescue
- C13, C14, C15, C20, C21, C23, C26, C33, C34: symbol lago_sch-rescue:C_Small -> lago_sch-rescue:C_Small-lago_sch-rescue
- C16: symbol lago_sch-rescue:CP1_Small -> lago_sch-rescue:CP1_Small-lago_sch-rescue
- C17, C18, C19, C24, C25, C35: symbol lago_sch-rescue:C -> lago_sch-rescue:C-lago_sch-rescue
- C27, C28, C29, C30, C31, C32: symbol lago_sch-rescue:CP_Small -> lago_sch-rescue:CP_Small-lago_sch-rescue
- D10, D9: symbol lago_sch-rescue:D_Schottky_Small_ALT -> lago_sch-rescue:D_Schottky_Small_ALT-lago_sch-rescue
- D7: symbol lago_sch-rescue:Led_Small -> lago_sch-rescue:Led_Small-lago_sch-rescue
- D8: symbol lago_sch-rescue:D_Schottky_Small -> lago_sch-rescue:D_Schottky_Small-lago_sch-rescue
- J3: symbol lago_sch-rescue:BARREL_JACK -> lago_sch-rescue:BARREL_JACK-lago_sch-rescue
- JP1, JP6: symbol lago_sch-rescue:Jumper_NO_Small -> lago_sch-rescue:Jumper_NO_Small-lago_sch-rescue
- JP7: symbol lago_sch-rescue:Jumper -> lago_sch-rescue:Jumper-lago_sch-rescue
- L1, L3, L4, L5, L6: symbol lago_sch-rescue:L -> lago_sch-rescue:L-lago_sch-rescue
- L2: symbol lago_sch-rescue:INDUCTOR_SMALL -> lago_sch-rescue:INDUCTOR_SMALL-lago_sch-rescue
- R21, R22, R24, R27, R29, R30: symbol lago_sch-rescue:R -> lago_sch-rescue:R-lago_sch-rescue
- R23, R25, R26, R28, R31, R32, R33, R34: symbol lago_sch-rescue:R_Small -> lago_sch-rescue:R_Small-lago_sch-rescue
- U2: symbol lago_sch-rescue:LM2596 -> lago_sch-rescue:LM2596-lago_sch-rescue
- U3: symbol lago_sch-rescue:LT8471 -> lago_sch-rescue:LT8471-lago_sch-rescue
- W11, W12, W13, W14: symbol lago_sch-rescue:TEST_1P -> lago_sch-rescue:TEST_1P-lago_sch-rescue
